File: Battery_Charger_Balancer_2/Battery_Charger_Balancer_2.kicad_sch (KiCad schematic)
At the start: 118 parts, among them J1 GSB1C41110SSHR, J2 Conn_02x03_Odd_Even, J3 Conn_01x06_Pin, J4 Conn_01x02_Socket, J5 Conn_01x02_Socket, J6 Conn_01x02_Pin, Q1 GSFD0646, SW1 SW_SPDT, U1 RT1719GQW, U10 BAV74_215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

Commit message: Updates after production of first rev
Parts:
- C16, C18, C20, C27, C31: value 10uF -> 4.7uF
- R13: value 13.7k -> 1.62k
- R2: value 453k -> 887k
- R25: now not fitted
Other:
- note added: "2.06A I_LIM"
- note added: "TABLE_SEL = 1, PSEL1 = 100, PSEL2 = 001 USB_SET set for "No USB Ability" PATH_OPT set to enable FET when PDO matches ADDR set to 0x43"
- note removed: "2.43A I_LIM"
- note removed: "Note: Need to figure out proper R/C values for gate pin slew rate"
- note removed: "TABLE_SEL = 1, PSEL1 = 000, PSEL2 = 001 USB_SET set for "No USB Ability" PATH_OPT set to enable FET when PDO matches ADDR set to 0x43"
Changed lines of the file:
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@@
 		)
 	)
-	(text "Note: Need to figure out proper R/C values for gate pin slew rate"
-		(exclude_from_sim no)
-		(at 166.116 14.478 0)
-		(effects
-			(font
-				(size 1.27 1.27)
-			)
-		)
-	)
-	(text "2.43A I_LIM"
+	(text "2.06A I_LIM"
 		(exclude_from_sim no)
 		(at 114.046 153.67 0)
@@
 		)
 	)
-	(text "TABLE_SEL = 1, PSEL1 = 000, PSEL2 = 001\nUSB_SET set for \"No USB Ability\"\nPATH_OPT set to enable FET when PDO matches\nADDR set to 0x43"
+	(text "TABLE_SEL = 1, PSEL1 = 100, PSEL2 = 001\nUSB_SET set for \"No USB Ability\"\nPATH_OPT set to enable FET when PDO matches\nADDR set to 0x43"
 		(exclude_from_sim no)
 		(at 122.936 85.344 0)
@@
 			)
 		)
-		(property "Value" "10uF"
+		(property "Value" "4.7uF"
 			(at 388.62 55.8799 0)
 			(show_name no)
@@
 			)
 		)
-		(property "Value" "13.7k"
+		(property "Value" "1.62k"
 			(at 118.11 149.8599 0)
 			(show_name no)
@@
 			)
 		)
-		(property "Value" "10uF"
+		(property "Value" "4.7uF"
 			(at 388.62 40.6399 0)
 			(show_name no)
@@
 			)
 		)
-		(property "Value" "10uF"
+		(property "Value" "4.7uF"
 			(at 388.62 114.2999 0)
 			(show_name no)
@@
 			)
 		)
-		(property "Value" "10uF"
+		(property "Value" "4.7uF"
 			(at 388.62 143.5099 0)
 			(show_name no)
@@
 			)
 		)
-		(property "Value" "453k"
+		(property "Value" "887k"
 			(at 102.87 73.6599 0)
 			(show_name no)
@@
 			)
 		)
-		(property "Value" "10uF"
+		(property "Value" "4.7uF"
 			(at 388.62 85.0899 0)
 			(show_name no)
@@
 		(on_board yes)
 		(in_pos_files yes)
-		(dnp no)
+		(dnp yes)
 		(fields_autoplaced yes)
 		(property "Reference" "R25"

Commit message: Finial version of the original design
Parts:
- R2: value 887k -> 887k (909k)
- R38: value 11k -> 11k (10k)
Other:
- moved on the sheet: D1, R28, R3, R5
Changed lines of the file:
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@@
 	(wire
 		(pts
-			(xy 92.71 76.2) (xy 92.71 77.47)
+			(xy 90.17 57.15) (xy 90.17 58.42)
 		)
 		(stroke
@@
 	(wire
 		(pts
-			(xy 92.71 46.99) (xy 92.71 68.58)
+			(xy 90.17 46.99) (xy 90.17 49.53)
 		)
 		(stroke
@@
 	(wire
 		(pts
-			(xy 74.93 40.64) (xy 74.93 49.53)
+			(xy 68.58 40.64) (xy 68.58 49.53)
 		)
 		(stroke
@@
 	(wire
 		(pts
-			(xy 120.65 46.99) (xy 92.71 46.99)
+			(xy 120.65 46.99) (xy 90.17 46.99)
 		)
 		(stroke
@@
 	(wire
 		(pts
-			(xy 83.82 77.47) (xy 83.82 68.58)
-		)
-		(stroke
-			(width 0)
-			(type default)
-		)
-	)
-	(wire
-		(pts
 			(xy 200.66 40.64) (xy 195.58 40.64)
 		)
@@
 	(wire
 		(pts
-			(xy 83.82 44.45) (xy 120.65 44.45)
+			(xy 77.47 44.45) (xy 120.65 44.45)
 		)
 		(stroke
@@
 	(wire
 		(pts
+			(xy 77.47 64.77) (xy 77.47 67.31)
+		)
+		(stroke
+			(width 0)
+			(type default)
+		)
+	)
+	(wire
+		(pts
 			(xy 176.53 128.27) (xy 176.53 130.81)
 		)
@@
 	(wire
 		(pts
-			(xy 95.25 40.64) (xy 74.93 40.64)
+			(xy 95.25 40.64) (xy 68.58 40.64)
 		)
 		(stroke
@@
 	(wire
 		(pts
-			(xy 83.82 53.34) (xy 83.82 44.45)
+			(xy 77.47 49.53) (xy 77.47 44.45)
 		)
 		(stroke
@@
 	(wire
 		(pts
-			(xy 97.79 49.53) (xy 97.79 77.47)
+			(xy 97.79 49.53) (xy 97.79 58.42)
 		)
 		(stroke
@@
 	(symbol
 		(lib_id "power:GND")
-		(at 83.82 77.47 0)
+		(at 77.47 67.31 0)
 		(unit 1)
 		(body_style 1)
@@
 		(fields_autoplaced yes)
 		(property "Reference" "#PWR04"
-			(at 83.82 83.82 0)
+			(at 77.47 73.66 0)
 			(hide yes)
 			(show_name no)
@@
 		)
 		(property "Value" "GND"
-			(at 83.82 82.55 0)
+			(at 77.47 72.39 0)
 			(show_name no)
 			(do_not_autoplace no)
@@
 		)
 		(property "Footprint" ""
-			(at 83.82 77.47 0)
+			(at 77.47 67.31 0)
 			(hide yes)
 			(show_name no)
@@
 		)
 		(property "Datasheet" ""
-			(at 83.82 77.47 0)
+			(at 77.47 67.31 0)
 			(hide yes)
 			(show_name no)
@@
 		)
 		(property "Description" "Power symbol creates a global label with name \"GND\" , ground"
-			(at 83.82 77.47 0)
+			(at 77.47 67.31 0)
 			(hide yes)
 			(show_name no)
@@
 	(symbol
 		(lib_id "Device:LED")
-		(at 83.82 64.77 270)
+		(at 77.47 60.96 270)
 		(mirror x)
 		(unit 1)
@@
 		(dnp no)
 		(property "Reference" "D1"
-			(at 87.63 66.04 90)
+			(at 81.28 62.23 90)
 			(show_name no)
 			(do_not_autoplace no)
@@
 		)
 		(property "Value" "LED"
-			(at 87.63 63.5 90)
+			(at 81.28 59.69 90)
 			(show_name no)
 			(do_not_autoplace no)
@@
 		)
 		(property "Footprint" "LED_SMD:LED_0603_1608Metric_Pad1.05x0.95mm_HandSolder"
-			(at 83.82 64.77 0)
+			(at 77.47 60.96 0)
 			(hide yes)
 			(show_name no)
@@
 		)
 		(property "Datasheet" ""
-			(at 83.82 64.77 0)
+			(at 77.47 60.96 0)
 			(hide yes)
 			(show_name no)
@@
 		)
 		(property "Description" "Light emitting diode"
-			(at 83.82 64.77 0)
+			(at 77.47 60.96 0)
 			(hide yes)
 			(show_name no)
@@
 		)
 		(property "Sim.Pins" "1=K 2=A"
-			(at 83.82 64.77 0)
+			(at 77.47 60.96 0)
 			(hide yes)
 			(show_name no)
@@
 	(symbol
 		(lib_id "Device:R")
-		(at 92.71 72.39 0)
+		(at 90.17 53.34 0)
 		(mirror x)
 		(unit 1)
@@
 		(dnp no)
 		(property "Reference" "R3"
-			(at 90.17 71.1199 0)
+			(at 87.63 52.0699 0)
 			(show_name no)
 			(do_not_autoplace no)
@@
 		)
 		(property "Value" "0"
-			(at 90.17 73.6599 0)
+			(at 87.63 54.6099 0)
 			(show_name no)
 			(do_not_autoplace no)
@@
 		)
 		(property "Footprint" "Resistor_SMD:R_0603_1608Metric_Pad0.98x0.95mm_HandSolder"
-			(at 90.932 72.39 90)
+			(at 88.392 53.34 90)
 			(hide yes)
 			(show_name no)
@@
 		)
 		(property "Datasheet" ""
-			(at 92.71 72.39 0)
+			(at 90.17 53.34 0)
 			(hide yes)
 			(show_name no)
@@
 		)
 		(property "Description" "Resistor"
-			(at 92.71 72.39 0)
+			(at 90.17 53.34 0)
 			(hide yes)
 			(show_name no)
@@
 	(symbol
 		(lib_id "power:GND")
-		(at 74.93 57.15 0)
+		(at 68.58 57.15 0)
 		(unit 1)
 		(body_style 1)
@@
 		(fields_autoplaced yes)
 		(property "Reference" "#PWR03"
-			(at 74.93 63.5 0)
+			(at 68.58 63.5 0)
 			(hide yes)
 			(show_name no)
@@
 		)
 		(property "Value" "GND"
-			(at 74.93 62.23 0)
+			(at 68.58 62.23 0)
 			(show_name no)
 			(do_not_autoplace no)
@@
 		)
 		(property "Footprint" ""
-			(at 74.93 57.15 0)
+			(at 68.58 57.15 0)
 			(hide yes)
 			(show_name no)
@@
 		)
 		(property "Datasheet" ""
-			(at 74.93 57.15 0)
+			(at 68.58 57.15 0)
 			(hide yes)
 			(show_name no)
@@
 		)
 		(property "Description" "Power symbol creates a global label with name \"GND\" , ground"
-			(at 74.93 57.15 0)
+			(at 68.58 57.15 0)
 			(hide yes)
 			(show_name no)
@@
 			)
 		)
-		(property "Value" "887k"
+		(property "Value" "887k (909k)"
 			(at 102.87 73.6599 0)
 			(show_name no)
@@
 	(symbol
 		(lib_id "Device:R")
-		(at 83.82 57.15 180)
+		(at 77.47 53.34 180)
 		(unit 1)
 		(body_style 1)
@@
 		(dnp no)
 		(property "Reference" "R5"
-			(at 87.63 56.134 0)
+			(at 81.28 52.324 0)
 			(show_name no)
 			(do_not_autoplace no)
@@
 		)
 		(property "Value" "2.2k"
-			(at 88.392 58.42 0)
+			(at 82.042 54.61 0)
 			(show_name no)
 			(do_not_autoplace no)
@@
 		)
 		(property "Footprint" "Resistor_SMD:R_0603_1608Metric_Pad0.98x0.95mm_HandSolder"
-			(at 85.598 57.15 90)
+			(at 79.248 53.34 90)
 			(hide yes)
 			(show_name no)
@@
 		)
 		(property "Datasheet" ""
-			(at 83.82 57.15 0)
+			(at 77.47 53.34 0)
 			(hide yes)
 			(show_name no)
@@
 		)
 		(property "Description" "Resistor"
-			(at 83.82 57.15 0)
+			(at 77.47 53.34 0)
 			(hide yes)
 			(show_name no)
@@
 	(symbol
 		(lib_id "power:GND")
-		(at 92.71 77.47 0)
+		(at 90.17 58.42 0)
 		(unit 1)
 		(body_style 1)
@@
 		(fields_autoplaced yes)
 		(property "Reference" "#PWR07"
-			(at 92.71 83.82 0)
+			(at 90.17 64.77 0)
 			(hide yes)
 			(show_name no)
@@
 		)
 		(property "Value" "GND"
-			(at 92.71 82.55 0)
+			(at 90.17 63.5 0)
 			(show_name no)
 			(do_not_autoplace no)
@@
 		)
 		(property "Footprint" ""
-			(at 92.71 77.47 0)
+			(at 90.17 58.42 0)
 			(hide yes)
 			(show_name no)
@@
 		)
 		(property "Datasheet" ""
-			(at 92.71 77.47 0)
+			(at 90.17 58.42 0)
 			(hide yes)
 			(show_name no)
@@
 		)
 		(property "Description" "Power symbol creates a global label with name \"GND\" , ground"
-			(at 92.71 77.47 0)
+			(at 90.17 58.42 0)
 			(hide yes)
 			(show_name no)
@@
 	(symbol
 		(lib_id "Device:R")
-		(at 74.93 53.34 0)
+		(at 68.58 53.34 0)
 		(unit 1)
 		(body_style 1)
@@
 		(fields_autoplaced yes)
 		(property "Reference" "R28"
-			(at 77.47 52.0699 0)
+			(at 71.12 52.0699 0)
 			(show_name no)
 			(do_not_autoplace no)
@@
 		)
 		(property "Value" "10k"
-			(at 77.47 54.6099 0)
+			(at 71.12 54.6099 0)
 			(show_name no)
 			(do_not_autoplace no)
@@
 		)
 		(property "Footprint" "Resistor_SMD:R_0603_1608Metric_Pad0.98x0.95mm_HandSolder"
-			(at 73.152 53.34 90)
+			(at 66.802 53.34 90)
 			(hide yes)
 			(show_name no)
@@
 		)
 		(property "Datasheet" ""
-			(at 74.93 53.34 0)
+			(at 68.58 53.34 0)
 			(hide yes)
 			(show_name no)
@@
 		)
 		(property "Description" "Resistor"
-			(at 74.93 53.34 0)
+			(at 68.58 53.34 0)
 			(hide yes)
 			(show_name no)
@@
 			)
 		)
-		(property "Value" "11k"
+		(property "Value" "11k (10k)"
 			(at 104.14 179.0699 0)
 			(show_name no)
@@
 	(symbol
 		(lib_id "power:GND")
-		(at 97.79 77.47 0)
+		(at 97.79 58.42 0)
 		(unit 1)
 		(body_style 1)
@@
 		(fields_autoplaced yes)
 		(property "Reference" "#PWR05"
-			(at 97.79 83.82 0)
+			(at 97.79 64.77 0)
 			(hide yes)
 			(show_name no)
@@
 		)
 		(property "Value" "GND"
-			(at 97.79 82.55 0)
+			(at 97.79 63.5 0)
 			(show_name no)
 			(do_not_autoplace no)
@@
 		)
 		(property "Footprint" ""
-			(at 97.79 77.47 0)
+			(at 97.79 58.42 0)
 			(hide yes)
 			(show_name no)
@@
 		)
 		(property "Datasheet" ""
-			(at 97.79 77.47 0)
+			(at 97.79 58.42 0)
 			(hide yes)
 			(show_name no)
@@
 		)
 		(property "Description" "Power symbol creates a global label with name \"GND\" , ground"
-			(at 97.79 77.47 0)
+			(at 97.79 58.42 0)
 			(hide yes)
 			(show_name no)
